File: Eagle design files/electronicload3.00.brd (EAGLE design)
At the start: 72 x 59 mm, 36 parts, among them IC1 MCP6072-E/SN, J1 ZX62D-B-5PA8, Q1 BTS133BKSA1, U1 ELECTRONICLOAD_ARDUINO_BLUEPI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, U2 MCP4725, X1 ED350/2

Commit message: Corrected BOM and eagle files before devices are manufactured
Parts:
- C5: value 1u -> 10n
- C7: value 1u -> 100pF
Changed lines of the file:
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@@
 <attribute name="VOLTAGE" value="16V" x="9.3" y="7" size="1.778" layer="27" rot="R90" display="off"/>
 </element>
-<element name="C7" library="rcl" library_urn="urn:adsk.eagle:library:334" package="C0603K" package3d_urn="urn:adsk.eagle:package:23680/2" value="1u" x="23" y="20.04" smashed="yes" rot="R270">
+<element name="C7" library="rcl" library_urn="urn:adsk.eagle:library:334" package="C0603K" package3d_urn="urn:adsk.eagle:package:23680/2" value="100pF" x="23" y="20.04" smashed="yes" rot="R270">
 <attribute name="DIGIKEY" value="445-7456-1-ND" x="23" y="20.04" size="1.778" layer="27" rot="R270" display="off"/>
 <attribute name="NAME" x="23.55" y="21.66" size="1.016" layer="25" font="vector" ratio="17" rot="R90"/>
@@
 <attribute name="VALUE" x="25.765" y="11.195" size="1.27" layer="27"/>
 </element>
-<element name="C5" library="rcl" library_urn="urn:adsk.eagle:library:334" package="C0603K" package3d_urn="urn:adsk.eagle:package:23680/2" value="1u" x="24.1" y="12.2" smashed="yes" rot="R90">
+<element name="C5" library="rcl" library_urn="urn:adsk.eagle:library:334" package="C0603K" package3d_urn="urn:adsk.eagle:package:23680/2" value="10n" x="24.1" y="12.2" smashed="yes" rot="R90">
 <attribute name="DIGIKEY" value="445-7456-1-ND" x="24.1" y="12.2" size="1.778" layer="27" rot="R90" display="off"/>
 <attribute name="NAME" x="24.55" y="8.7" size="1.016" layer="25" ratio="17" rot="R90"/>
