File: Eagle design files/electronicload3.00.sch (EAGLE design)
At the start: 36 parts, among them IC1 MCP6072-E/SN, J1 ZX62D-B-5PA8, Q1 BTS133BKSA1, U1 ELECTRONICLOAD_ARDUINO_BLUEPI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, U2 MCP4725, X1 ED350/2

Commit message: Corrected BOM and eagle files before devices are manufactured
Parts:
- C5: value 1u -> 10n
- C7: value 1u -> 100pF
Changed lines of the file:
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@@
 <part name="GND8" library="supply1" library_urn="urn:adsk.eagle:library:371" deviceset="GND" device=""/>
 <part name="GND7" library="supply1" library_urn="urn:adsk.eagle:library:371" deviceset="GND" device=""/>
-<part name="C7" library="rcl" library_urn="urn:adsk.eagle:library:334" deviceset="C-EU" device="C0603K" package3d_urn="urn:adsk.eagle:package:23680/2" value="1u">
+<part name="C7" library="rcl" library_urn="urn:adsk.eagle:library:334" deviceset="C-EU" device="C0603K" package3d_urn="urn:adsk.eagle:package:23680/2" value="100pF">
 <spice>
 <pinmapping spiceprefix="C">
@@
 <attribute name="DIGIKEY" value="RMCF0603JT150RCT-ND"/>
 </part>
-<part name="C5" library="rcl" library_urn="urn:adsk.eagle:library:334" deviceset="C-EU" device="C0603K" package3d_urn="urn:adsk.eagle:package:23680/2" value="1u">
+<part name="C5" library="rcl" library_urn="urn:adsk.eagle:library:334" deviceset="C-EU" device="C0603K" package3d_urn="urn:adsk.eagle:package:23680/2" value="10n">
 <spice>
 <pinmapping spiceprefix="C">
@@
 <attribute name="DIGIKEY" x="105.41" y="45.72" size="1.778" layer="96" display="off"/>
 </instance>
-<instance part="C5" gate="G$1" x="96.52" y="40.64" rot="R180">
+<instance part="C5" gate="G$1" x="96.52" y="40.64" smashed="yes" rot="R180">
 <attribute name="DIGIKEY" x="96.52" y="40.64" size="1.778" layer="96" rot="R180" display="off"/>
 <attribute name="TEMPCOEFF" x="96.52" y="40.64" size="1.778" layer="96" rot="R180" display="off"/>
 <attribute name="TOLERANCE" x="96.52" y="40.64" size="1.778" layer="96" rot="R180" display="off"/>
 <attribute name="VOLTAGE" x="96.52" y="40.64" size="1.778" layer="96" rot="R180" display="off"/>
+<attribute name="NAME" x="91.694" y="38.481" size="1.778" layer="95"/>
+<attribute name="VALUE" x="98.044" y="38.481" size="1.778" layer="96"/>
 </instance>
 <instance part="GND9" gate="1" x="96.52" y="34.29"/>
